File: hardware/Qwiic2PinHeaders/Qwiic2PinHeaders.kicad_pcb (KiCad board)
At the start: 2 copper layers, 10 x 25 mm, 4 parts, among them J1 Conn_01x04_Pin, J2 Qwiic, J3 Qwiic

Commit message: hardware: minor tweaks
Other:
- board text added: "Qwiic to PinHeaders"
- board text removed: "Quiic to PinHeaders"
Changed lines of the file:
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@@
 		)
 	)
-	(gr_text "Quiic\nto\nPinHeaders"
-		(at 145 46.1 0)
+	(gr_text "Qwiic\nto\nPinHeaders"
+		(at 145.05 45.85 0)
 		(layer "B.SilkS")
 		(effects

Commit message: hardware: add misc project files
Other:
- outline, holes or cut-outs redrawn
