File: hardware/USON2SOIC-8/USON2SOIC-8.kicad_pcb (KiCad board)
At the start: 2 copper layers, 9.3 x 5.9 mm, 2 parts, among them U1 W25Q16JVUXIQ, U2 W25Q32JVSS

Commit message: hardware: add misc project files
Routing:
- net GND: track 4.62 -> 5.47 mm
Other:
- outline, holes or cut-outs redrawn
