File: hardware/TommyDSP/MCU-Core.kicad_sch (KiCad schematic)
At the start: 32 parts, among them SW201 SW_Push, SW202 SW_Push, U201 W25Q128JVS, U202 DNF, U203 RP2350_60QFN, Y201 ABM8-272-T3

Commit message: hardware: minor tweaks
Other:
- note added: "Optional Secondary flash or PSRAM (U201), using the second chip select (XIP_SS_N[1]) on GPIO0. N.B. Pull-up R202 will be required as GPIOs default to pull-downs at power-up."
- note removed: "Optional Secondary flash or PSRAM (U201), using the second chip select (XIP_SS_N[1]) on GPIO0. N.B. Pull-up R204 will be required as GPIOs default to pull-downs at power-up."
Changed lines of the file:
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@@
 		)
 	)
-	(text "Optional Secondary flash or PSRAM (U201), using the second chip select (XIP_SS_N[1]) on GPIO0.\nN.B. Pull-up R204 will be required as GPIOs default to pull-downs at power-up."
+	(text "Optional Secondary flash or PSRAM (U201), using the second chip select (XIP_SS_N[1]) on GPIO0.\nN.B. Pull-up R202 will be required as GPIOs default to pull-downs at power-up."
 		(exclude_from_sim no)
 		(at 15.494 197.104 0)

Commit message: hardware: add misc project files
Changed lines of the file:
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@@
+	(wire
+		(pts
+			(xy 137.16 50.8) (xy 147.32 50.8)
+		)
+		(stroke
+			(width 0)
+			(type default)
+		)
+	)
 	(wire
 		(pts
@@
 		(pts
 			(xy 194.31 41.91) (xy 198.12 41.91)
-		)
-		(stroke
-			(width 0)
-			(type default)
-		)
-	)
-	(wire
-		(pts
-			(xy 137.16 50.8) (xy 147.32 50.8)
 		)
 		(stroke
@@
 	)
 	(label "VREG_AVDD"
-		(at 137.795 50.8 0)
-		(effects
-			(font
+		(at 137.16 50.8 0)
+		(effects
+			(font

Commit message: bump to KiCad V10, add logo
Other:
- title: MCU Core -> TommyDSP
