File: hardware/TommyDSP/Peripherals.kicad_sch (KiCad schematic)
At the start: 39 parts, among them J501 USB_C_Receptacle_USB2.0_16P, J502 AudioJack3_SwitchTR, J503 XH-2.50mm Horizontal, J504 AudioJack3_SwitchTR, J505 EXT.IN, J506 AudioJack3_SwitchTR, J507 XH-2.50mm Horizontal, J508 EXT.OUT, J509 Conn_01x03_Pin, J510 AudioJack3_SwitchTR, J511 Micro_SD_Card_Det1, J512 Qwiic, SW501 RotaryEncoder_Switch_MP

Commit message: bump to KiCad V10, add logo
Parts:
- RV501, RV502, RV503: footprint Potentiometer_THT:Potentiometer_Alps_RK09K_Single_Vertical -> Project:Potentiometer_Alps_RK09K_Single_Vertical
Other:
- title: Peripherals -> TommyDSP
